Commit message: Add files via upload

File: rw/urdf/rw_bot.urdf (robot description, URDF)
Before this commit: robot rw_bot, 17 links, 16 joints
Links:
- removed link laser_frame
- removed link lidar_link_optical
- added link front_laser_frame; collision mesh filename=file://$(find rw)/robot_meshes/front_lidar.stl; visual mesh filename=file://$(find rw)/robot_meshes/front_lidar.stl
- added link front_lidar_link_optical
Joints:
- joint front_camera_optical_joint: origin xyz=0.0202968 0 0.0228071 rpy=${pi} -${pi} -${pi} -> xyz=0.0202968 0 0.0228071 rpy=0.0 0.0 0.0
- joint laser_joint: child laser_frame -> front_laser_frame
- joint lidar_optical_joint: child lidar_link_optical -> front_lidar_link_optical; origin xyz=0.025 0 0.03 rpy=${pi} -${pi} -${pi} -> xyz=0.025 0 0.03 rpy=0.0 0.0 0.0; parent laser_frame -> front_laser_frame
